Commit message: realsense gazebo plugin working, creating operational mobile manipulator in progress

File: src/mobile-platform/urdf/mobile-platform.urdf.xacro (robot description, xacro)
@@ -1,12 +1,6 @@
 <?xml version="1.0"?>
 <robot name="mobile_platform" xmlns:xacro="http://www.ros.org/wiki/xacro">
-  <!-- includes -->
   <xacro:include filename="$(find dingo_description)/urdf/dingo.urdf.xacro"/>
-  <xacro:include filename="$(find moveit_resources_panda_description)/urdf/panda_arm_hand.urdf.xacro"/>
-  <!-- coś mi nie działa kurwa z przekazywaniem parametetrów więc musiałem zdefiniować je na sztywno w panda_arm_hand.xacro -->
-  <!-- <joint name="dingo_panda_joint" type="fixed">
-    <parent link="base_link"/>
-    <child link="panda_link0"/>
-    <origin xyz="0 0 0.1"/>
-  </joint> -->
+  <xacro:include filename="$(find franka_description)/robots/panda/panda.urdf.xacro"/>
+  <xacro:include filename="$(find packagename)/urdf/urdf_d435.gazebo.xacro"/>
 </robot>

Commit message: developing slam with dingo

File: src/mobile-platform/urdf/mobile-platform.urdf.xacro (robot description, xacro)
@@ -2,5 +2,17 @@
 <robot name="mobile_platform" xmlns:xacro="http://www.ros.org/wiki/xacro">
   <xacro:include filename="$(find dingo_description)/urdf/dingo.urdf.xacro"/>
-  <xacro:include filename="$(find franka_description)/robots/panda/panda.urdf.xacro"/>
-  <xacro:include filename="$(find packagename)/urdf/urdf_d435.gazebo.xacro"/>
+  <!-- <xacro:include filename="$(find franka_description)/robots/panda/panda.urdf.xacro"/> -->
+  <!-- <xacro:include filename="$(find mobile-platform)/urdf/_d435.urdf.xacro"/> -->
+  <!-- <xacro:sensor_d435 parent="panda_link8">
+    <origin xyz="0.035 -0.035 0.05" rpy="0 -1.57 -0.785"/>
+  </xacro:sensor_d435> -->
+  <xacro:include filename="$(find mobile-platform)/urdf/_d435.urdf.xacro"/>
+  <xacro:sensor_d435 parent="base_link" topics_ns="camera_front">
+    <origin xyz="0.35  0 0.1" rpy="0 -0.13 0"/>
+  </xacro:sensor_d435>
+  <!-- <joint name="panda_base_joint" type="fixed">
+    <parent link="base_link"/>
+    <child link="panda_link0"/>
+    <origin xyz="0 0 0.1"/>
+  </joint> -->
 </robot>
