Commit message: added launch file with both platform and arm

File: src/mobile-platform/urdf/only_panda.urdf.xacro (robot description, xacro)
@@ -4,8 +4,8 @@
   <xacro:include filename="$(find mobile-platform)/urdf/_d435.urdf.xacro"/>
   <!-- <xacro:include filename="$(find mobile-platform)/urdf/_d435.gazebo.xacro"/> -->
-  <link name="world" />
-  <joint name="world_joint" type="fixed">
+  <link name="panda_base_link" />
+  <joint name="link_link_link" type="fixed">
     <origin xyz="0 0 0" rpy="0 0 0" />
-    <parent link="world" />
+    <parent link="panda_base_link" />
     <child  link="panda_link0" />
   </joint>

Commit message: repaired only_panda launch

File: src/mobile-platform/urdf/only_panda.urdf.xacro (robot description, xacro)
@@ -4,8 +4,8 @@
   <xacro:include filename="$(find mobile-platform)/urdf/_d435.urdf.xacro"/>
   <!-- <xacro:include filename="$(find mobile-platform)/urdf/_d435.gazebo.xacro"/> -->
-  <link name="panda_base_link" />
-  <joint name="link_link_link" type="fixed">
+  <link name="world" />
+  <joint name="world_joint" type="fixed">
     <origin xyz="0 0 0" rpy="0 0 0" />
-    <parent link="panda_base_link" />
+    <parent link="world" />
     <child  link="panda_link0" />
   </joint>
